Commit message: Added static calibration node and launcher

File: urdf/humanArm5.urdf (robot description, URDF)
Before this commit: robot humanArm5, 13 links, 12 joints
Joints:
- joint el_x: axis 0 0 1 -> 0 0 -1
- joint sh_y: axis 0 0 1 -> 0 0 -1

Commit message: Added OpenZen library example launch file

File: urdf/humanArm5.urdf (robot description, URDF)
Before this commit: robot humanArm5, 13 links, 12 joints
Joints:
- joint el_x: axis 0 0 -1 -> 0 0 1
- joint sh_y: axis 0 0 -1 -> 0 0 1

Commit message: Adapted nodes to new arm package name

File: urdf/humanArm5.urdf (robot description, URDF)
Before this commit: robot humanArm5, 13 links, 12 joints
Joints:
- joint sh_z: origin xyz=0 0 0 rpy=0 0 0 -> xyz=0 0 0 rpy=0 0 1.57079632679490

Commit message: Created generic node to cover all functionality though configuration

File: urdf/humanArm5.urdf (robot description, URDF)
Before this commit: robot humanArm5, 13 links, 12 joints
Joints:
- joint sh_z: origin xyz=0 0 0 rpy=0 0 1.57079632679490 -> xyz=0 0 0 rpy=0 0 0
